File: RaspiPowerHat.sch (EAGLE design)
At the start: 28 parts, among them U2 Value, U3 LM25011MYX/NOPB, X1 RASPI_GPIO_B+#_PIN

Commit message: Added another RGB channel, fixed footprints
Parts:
- added BLUE2, GREEN2, RED2: NTD4906N, transistor-power:4906N
- added C1: (no value), rcl:CPOL-USC
- added LED1: (no value), SparkFun-Connectors:M04JST-PTH-VERT
- U$15: value 16SVPC39MV -> B360A-13-F; device TI-LMR14050SSDA:16SVPC39MV -> TI-LMR14050SSDA:B360A-13-F
- renumbered B to BLUE, G to GREEN, R to RED
Connections:
- net GPIO17 renamed RED1
- net GPIO22 renamed GREEN1
- net GPIO24 renamed BLUE1
- new net BLUE2: BLUE2.D, LED1.4
- new net GREEN2: GREEN2.D, LED1.2
- new net INBLUE2: BLUE2.G, X1.SPI_MOSI
- new net INGREEN2: GREEN2.G, X1.SPI_SCLK
- new net INRED2: RED2.G, X1.SPI_MISO
- new net N$2: CON1-1.KL, U$15.A
- new net RED2: LED1.3, RED2.D
- net 12V: now also LED1.1
- net 24VIN: now also U$15.K; no longer CON1-1.KL
- net 5V: now also C1.+; no longer U$15.1
- net GND: now also BLUE2.SG1, C1.-, GREEN2.SG1, RED2.SG1; no longer U$15.2
